Commit message: WIP to refactored launch

File: yumi_description/urdf/Extras/yumi_optodaq_sensors.xacro (robot description, xacro)
@@ -3,5 +3,5 @@
   <xacro:macro name="yumi_optodaq_sensor" params="parent name *origin">
     <!--joint between {parent} and base-->
-    <joint name="${parent}_joint" type="fixed">
+    <joint name="${parent}_f_joint" type="fixed">
       <xacro:insert_block name="origin"/>
       <parent link="${parent}"/>
