Commit message: Set gripper transforms according to the balancing setup

File: yumi_description/urdf/yumi.urdf.xacro (robot description, xacro)
@@ -21,25 +21,17 @@
   </xacro:yumi>
  <xacro:yumi_optodaq_sensor name="optodaq_r" parent="yumi_link_7_r">
-   <origin xyz="0 0 0.033" rpy="0 0 ${5*PI/8}" />
- </xacro:yumi_optodaq_sensor>
- <xacro:yumi_optodaq_sensor name="optodaq_l" parent="yumi_link_7_l">
-   <origin xyz="0 0 0.033" rpy="0 ${PI} ${-PI/4}" />
- </xacro:yumi_optodaq_sensor>
- <!--right gripper-->
- <xacro:yumi_servo_gripper name="gripper_r" hardware_interface="hardware_interface/EffortJointInterface" parent="optodaq_r_sensor_link">
-   <origin xyz="0 0 0.033" rpy="${PI} 0.0 ${PI/4}" />
- </xacro:yumi_servo_gripper>
- <!--left gripper-->
- <xacro:yumi_servo_gripper name="gripper_l" hardware_interface="hardware_interface/EffortJointInterface" parent="optodaq_l_sensor_link">
-   <origin xyz="0 0 -0.033" rpy="${PI} 0.0 ${PI/4}" />
- </xacro:yumi_servo_gripper>
- <!-- Surface piece -->
- <xacro:yumi_fold_case name="fold_case" parent="gripper_r">
-   <origin xyz="0 0 0" rpy="0 0 0" />
- </xacro:yumi_fold_case>
- <!-- Rod piece -->
- <xacro:yumi_rod name="rod_piece" parent="gripper_l">
-   <origin xyz="0 0 0" rpy="0 0 0" />
- </xacro:yumi_rod>
+      <origin xyz="0 0 0.033" rpy="0 ${PI} 3.67" />
+  </xacro:yumi_optodaq_sensor>
+  <xacro:yumi_optodaq_sensor name="optodaq_l" parent="yumi_link_7_l">
+	  <origin xyz="0 0 0.033" rpy="0 ${PI} -1.9" />
+  </xacro:yumi_optodaq_sensor>
+<!--right gripper-->
+  <xacro:yumi_servo_gripper name="gripper_r" hardware_interface="hardware_interface/EffortJointInterface" parent="yumi_link_7_r">
+    <origin xyz="0 0 0.066" rpy="0.0 0.0 -3.948" />
+  </xacro:yumi_servo_gripper>
+  <!--left gripper-->
+  <xacro:yumi_servo_gripper name="gripper_l" hardware_interface="hardware_interface/EffortJointInterface" parent="yumi_link_7_l">
+    <origin xyz="0 0 0.066" rpy="0.0 0.0 0.818" />
+  </xacro:yumi_servo_gripper>
   <xacro:property name="yumi_setup" value="$(arg yumi_setup)" />
   <xacro:if value="${yumi_setup == 'robot_centric'}">

Commit message: Change args definition to be compatible with future ros

File: yumi_description/urdf/yumi.urdf.xacro (robot description, xacro)
@@ -11,4 +11,17 @@
   <!-- Import Gazebo plugins -->
   <xacro:include filename="$(find yumi_description)/urdf/Gazebo/gazebo.urdf.xacro"/>
+  <xacro:property name="yumi_setup" value="$(arg yumi_setup)" />
+  <xacro:if value="${yumi_setup == 'robot_centric'}">
+    <!-- Pure YuMi URDF, with no joints connecting it to any other robot or pedestal. Neither accessories. -->
+  </xacro:if>
+  <xacro:if value="${yumi_setup == 'default'}">
+    <xacro:property name="yumi_parent" value="world" />
+    <link name="world"/>
+    <joint name="world_joint" type="fixed">
+      <parent link="world"/>
+      <child link="yumi_base_link"/>
+      <origin xyz="0 0 0.1" rpy="0 0 0" />
+    </joint>
+  </xacro:if>
   <!--yumi-->
   <xacro:yumi name="yumi" hardware_interface="hardware_interface/$(arg arms_interface)" parent="${yumi_parent}" >
@@ -23,16 +36,3 @@
     <origin xyz="0 0 0.007" rpy="0 0 ${PI}" />
   </xacro:yumi_servo_gripper>
-  <xacro:property name="yumi_setup" value="$(arg yumi_setup)" />
-  <xacro:if value="${yumi_setup == 'robot_centric'}">
-  	<!-- Pure YuMi URDF, with no joints connecting it to any other robot or pedestal. Neither accessories. -->
-  </xacro:if>
-  <xacro:if value="${yumi_setup == 'default'}">
-    <xacro:property name="yumi_parent" value="world" />
-    <link name="world"/>
-    <joint name="world_joint" type="fixed">
-      <parent link="world"/>
-      <child link="yumi_base_link"/>
-      <origin xyz="0 0 0.1" rpy="0 0 0" />
-    </joint>
-  </xacro:if>
 </robot>

Commit message: Change args definition to be compatible with future ros

File: yumi_description/urdf/yumi.urdf.xacro (robot description, xacro)
@@ -13,4 +13,17 @@
   <!-- Import Gazebo plugins -->
   <xacro:include filename="$(find yumi_description)/urdf/Gazebo/gazebo.urdf.xacro"/>
+  <xacro:property name="yumi_setup" value="$(arg yumi_setup)" />
+  <xacro:if value="${yumi_setup == 'robot_centric'}">
+    <!-- Pure YuMi URDF, with no joints connecting it to any other robot or pedestal. Neither accessories. -->
+  </xacro:if>
+  <xacro:if value="${yumi_setup == 'default'}">
+    <xacro:property name="yumi_parent" value="world" />
+    <link name="world"/>
+    <joint name="world_joint" type="fixed">
+      <parent link="world"/>
+      <child link="yumi_base_link"/>
+      <origin xyz="0 0 0.1" rpy="0 0 0" />
+    </joint>
+  </xacro:if>
   <!--yumi-->
   <xacro:yumi name="yumi" hardware_interface="hardware_interface/$(arg arms_interface)" parent="${yumi_parent}" >
@@ -31,16 +44,3 @@
    <origin xyz="0 0 -0.033" rpy="${PI} 0.0 ${PI/4}" />
  </xacro:yumi_servo_gripper>
-  <xacro:property name="yumi_setup" value="$(arg yumi_setup)" />
-  <xacro:if value="${yumi_setup == 'robot_centric'}">
-  	<!-- Pure YuMi URDF, with no joints connecting it to any other robot or pedestal. Neither accessories. -->
-  </xacro:if>
-  <xacro:if value="${yumi_setup == 'default'}">
-    <xacro:property name="yumi_parent" value="world" />
-    <link name="world"/>
-    <joint name="world_joint" type="fixed">
-      <parent link="world"/>
-      <child link="yumi_base_link"/>
-      <origin xyz="0 0 0.1" rpy="0 0 0" />
-    </joint>
-  </xacro:if>
 </robot>

Commit message: Port extras for optodaq_sensor

File: yumi_description/urdf/yumi.urdf.xacro (robot description, xacro)
@@ -9,30 +9,38 @@
   <!--Import the yumi servo gripper macro -->
   <xacro:include filename="$(find yumi_description)/urdf/Grippers/yumi_servo_gripper.xacro"/>
+  <!--Import the yumi optodaq sensors macro -->
+  <xacro:include filename="$(find yumi_description)/urdf/Extras/yumi_optodaq_sensors.xacro"/>
   <!-- Import Gazebo plugins -->
   <xacro:include filename="$(find yumi_description)/urdf/Gazebo/gazebo.urdf.xacro"/>
+  <xacro:property name="yumi_setup" value="$(arg yumi_setup)" />
+  <xacro:if value="${yumi_setup == 'robot_centric'}">
+    <!-- Pure YuMi URDF, with no joints connecting it to any other robot or pedestal. Neither accessories. -->
+  </xacro:if>
+  <xacro:if value="${yumi_setup == 'default'}">
+  </xacro:if>
+  <xacro:property name="yumi_parent" value="world" />
+  <link name="world"/>
+  <joint name="world_joint" type="fixed">
+    <parent link="world"/>
+    <child link="yumi_base_link"/>
+    <origin xyz="0 0 0.1" rpy="0 0 0" />
+  </joint>
   <!--yumi-->
   <xacro:yumi name="yumi" hardware_interface="hardware_interface/$(arg arms_interface)" parent="${yumi_parent}" >
     <origin xyz="0 0 0.1" rpy="0 0 0" />
   </xacro:yumi>
-  <!--right gripper-->
-  <xacro:yumi_servo_gripper name="gripper_r" hardware_interface="hardware_interface/$(arg grippers_interface)" parent="yumi_link_7_r">
-    <origin xyz="0 0 0.007" rpy="0 0 ${PI}" />
+ <xacro:yumi_optodaq_sensor name="optodaq_r" parent="yumi_link_7_r">
+      <origin xyz="0 0 0.033" rpy="0 ${PI} 3.67" />
+  </xacro:yumi_optodaq_sensor>
+  <xacro:yumi_optodaq_sensor name="optodaq_l" parent="yumi_link_7_l">
+	  <origin xyz="0 0 0.033" rpy="0 ${PI} -1.9" />
+  </xacro:yumi_optodaq_sensor>
+<!--right gripper-->
+  <xacro:yumi_servo_gripper name="gripper_r" hardware_interface="hardware_interface/EffortJointInterface" parent="yumi_link_7_r">
+    <origin xyz="0 0 0.066" rpy="0.0 0.0 -3.948" />
   </xacro:yumi_servo_gripper>
   <!--left gripper-->
-  <xacro:yumi_servo_gripper name="gripper_l" hardware_interface="hardware_interface/$(arg grippers_interface)" parent="yumi_link_7_l">
-    <origin xyz="0 0 0.007" rpy="0 0 ${PI}" />
+  <xacro:yumi_servo_gripper name="gripper_l" hardware_interface="hardware_interface/EffortJointInterface" parent="yumi_link_7_l">
+    <origin xyz="0 0 0.066" rpy="0.0 0.0 0.818" />
   </xacro:yumi_servo_gripper>
-  <xacro:property name="yumi_setup" value="$(arg yumi_setup)" />
-  <xacro:if value="${yumi_setup == 'robot_centric'}">
-  	<!-- Pure YuMi URDF, with no joints connecting it to any other robot or pedestal. Neither accessories. -->
-  </xacro:if>
-  <xacro:if value="${yumi_setup == 'default'}">
-    <xacro:property name="yumi_parent" value="world" />
-    <link name="world"/>
-    <joint name="world_joint" type="fixed">
-      <parent link="world"/>
-      <child link="yumi_base_link"/>
-      <origin xyz="0 0 0.1" rpy="0 0 0" />
-    </joint>
-  </xacro:if>
 </robot>
